File: circuit/schematics/test_brd.sch (EAGLE design)
At the start: 1 part

Commit message: add some parts
Parts:
- added C1: 0.1μF, resistor:C-EU025-040X050
- added C2: 3.3μF, resistor:CPOL-EUE2.5-5
- added R1: 20kΩ, resistor:R-EU_0207/10
- added R2: 1kΩ, resistor:R-EU_0207/10
Changed lines of the file:
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@@
 <layer number="97" name="Info" color="7" fill="1" visible="yes" active="yes"/>
 <layer number="98" name="Guide" color="6" fill="1" visible="yes" active="yes"/>
+<layer number="99" name="SpiceOrder" color="5" fill="1" visible="yes" active="yes"/>
 </layers>
 <schematic xreflabel="%F%N/%S.%C%R" xrefpart="/%S.%C%R">
@@
 <parts>
 <part name="U$1" library="ESP32-DEVKITC" deviceset="ESP32DEVKITC" device=""/>
+<part name="R1" library="resistor" library_urn="urn:adsk.eagle:library:348" deviceset="R-EU_" device="0207/10" package3d_urn="urn:adsk.eagle:package:25939/1" value="20kΩ"/>
+<part name="R2" library="resistor" library_urn="urn:adsk.eagle:library:348" deviceset="R-EU_" device="0207/10" package3d_urn="urn:adsk.eagle:package:25939/1" value="1kΩ"/>
+<part name="C1" library="resistor" library_urn="urn:adsk.eagle:library:348" deviceset="C-EU" device="025-040X050" package3d_urn="urn:adsk.eagle:package:26150/1" value="0.1μF"/>
+<part name="C2" library="resistor" library_urn="urn:adsk.eagle:library:348" deviceset="CPOL-EU" device="E2.5-5" package3d_urn="urn:adsk.eagle:package:25841/1" value="3.3μF"/>
 </parts>
 <sheets>
@@
 <instance part="U$1" gate="G$1" x="48.26" y="55.88" smashed="yes" rot="R90">
 <attribute name="NAME" x="43.18" y="29.21" size="1.27" layer="95" rot="R180"/>
+</instance>
+<instance part="R1" gate="G$1" x="78.74" y="86.36" smashed="yes">
+<attribute name="NAME" x="74.93" y="87.8586" size="1.778" layer="95"/>
+<attribute name="VALUE" x="74.93" y="83.058" size="1.778" layer="96"/>
+</instance>
+<instance part="R2" gate="G$1" x="78.74" y="76.2" smashed="yes">
+<attribute name="NAME" x="74.93" y="77.6986" size="1.778" layer="95"/>
+<attribute name="VALUE" x="74.93" y="72.898" size="1.778" layer="96"/>
+</instance>
+<instance part="C1" gate="G$1" x="78.74" y="63.5" smashed="yes">
+<attribute name="NAME" x="80.264" y="63.881" size="1.778" layer="95"/>
+<attribute name="VALUE" x="80.264" y="58.801" size="1.778" layer="96"/>
+</instance>
+<instance part="C2" gate="G$1" x="78.74" y="50.8" smashed="yes" rot="R180">
+<attribute name="NAME" x="77.597" y="50.3174" size="1.778" layer="95" rot="R270"/>
+<attribute name="VALUE" x="77.597" y="55.3974" size="1.778" layer="96" rot="R180"/>
 </instance>
 </instances>
@@
 </schematic>
 </drawing>
+<compatibility>
+<note version="8.2" severity="warning">
+Since Version 8.2, EAGLE supports online libraries. The ids
+of those online libraries will not be understood (or retained)
+with this version.
+</note>
+<note version="8.3" severity="warning">
+Since Version 8.3, EAGLE supports URNs for individual library
+assets (packages, symbols, and devices). The URNs of those assets
+will not be understood (or retained) with this version.
+</note>
+<note version="8.3" severity="warning">
+Since Version 8.3, EAGLE supports the association of 3D packages
+with devices in libraries, schematics, and board files. Those 3D
+packages will not be understood (or retained) with this version.
+</note>
+</compatibility>
 </eagle>

Commit message: dekita
Parts:
- added IC1: (no value), v-reg:78XXS
- added Q1: 2N5484, transistor-fet:2N5484
- added SV1, SV2: (no value), con-lsta:FE20-1
- added X1, X2: JST-XH-02-PIN-LONG-PAD, Rembrandt Electronics - JST XH Connectors v1-0:JST-XH-02-PIN-LONG-PAD
- added X3: JST-XH-05-PIN-LONG-PAD, Rembrandt Electronics - JST XH Connectors v1-0:JST-XH-05-PIN-LONG-PAD
- R1: value 20kΩ -> 10kΩ
- R2: value 1kΩ -> 330Ω
Connections:
- new net N$1: C1.1, IC1.IN, X1-1.S, X3-4.S
- new net N$2: C2.+, IC1.OUT, SV2.19
- new net N$3: C1.2, C2.-, IC1.GND, Q1.S, R1.1, SV2.14, X2-2.S, X3-3.S
- new net N$4: Q1.G, R1.2, R2.2
- new net N$5: R2.1, SV2.9
- new net N$6: X1-2.S, X2-1.S
- new net N$7: SV2.1, X3-1.S
- new net N$8: SV1.13, X3-2.S
- new net N$9: Q1.D, X3-5.S
Other:
- moved on the sheet: C1, C2, R1, R2, U$1
