File: circuit/schematics/test_brd_add_gnd.brd (EAGLE design)
At the start: 160 x 100 mm, 12 parts, among them Q1 2N5484, X1 JST-XH-02-PIN-LONG-PAD, X2 JST-XH-02-PIN-LONG-PAD, X3 JST-XH-05-PIN-LONG-PAD

Commit message: 整理された配線
Parts:
- moved R2 66.8 mm to (34.2, 58.6)
- moved IC1 50.1 mm to (8.85, 58.3)
- moved R1 50.0 mm to (27.9, 51.6)
- moved C2 33.3 mm to (11.3, 46.7), turned to 180 degrees
- moved C1 26.7 mm to (9.83, 63.1), turned to 270 degrees
- moved Q1 26.2 mm to (45.8, 57.8), turned to 270 degrees
- moved U$1 14.8 mm to (-39.6, 31.6)
- moved X1 7.31 mm to (-0.96, 62.9)
- moved X2 6.88 mm to (-0.90, 51.6)
- moved X3 4.12 mm to (72.5, 57.1)
Routing:
- net GND: track 0.00 -> 108.5 mm
- net N$1: track 0.00 -> 103.0 mm
- net N$8: track 0.00 -> 40.4 mm
- net N$2: track 0.00 -> 31.4 mm
- net N$5: track 0.00 -> 29.7 mm
- net N$9: track 0.00 -> 27.5 mm
- net N$7: track 0.00 -> 23.4 mm
- net N$4: track 0.00 -> 20.8 mm
- net N$6: track 0.00 -> 9.39 mm
Other:
- board size 160 x 100 mm -> 176 x 106 mm
