File: circuit/schematics/test_brd_add_gnd.brd (EAGLE design)
At the start: 81 x 29 mm, 12 parts, among them Q1 2N5484, X1 JST-XH-02-PIN-LONG-PAD, X2 JST-XH-02-PIN-LONG-PAD, X3 JST-XH-05-PIN-LONG-PAD

Commit message: drc cleared
Parts:
- removed U$1: ESP32DEVKITC, ESP32-DEVKITC:ESP32-DEVKITC
