File: circuit/schematics/cotroler.brd (EAGLE design)
At the start: 64.8 x 64.4 mm, 17 parts

Commit message: drc cleared
Parts:
- removed U$1: ESP32DEVKITC, ESP32-DEVKITC:ESP32-DEVKITC
Connections:
- net GND: no longer U$1.19, U$1.38
Changed lines of the file:
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@@
 <attribute name="VALUE" x="117.9576" y="78.9559" size="1.27" layer="27" ratio="10" rot="R180"/>
-</element>
-<element name="U$1" library="ESP32-DEVKITC" package="ESP32-DEVKITC" value="ESP32DEVKITC" x="289.56" y="168.91" smashed="yes">
-<attribute name="NAME" x="265.43" y="182.88" size="1.27" layer="21"/>
 </element>
 <element name="R6" library="resistor" library_urn="urn:adsk.eagle:library:348" package="0207/10" package3d_urn="urn:adsk.eagle:package:25939/1" value="" x="67.31" y="41.91" smashed="yes" rot="R90">
@@
 <contactref element="C3" pad="-"/>
 <contactref element="IC2" pad="GND"/>
-<contactref element="U$1" pad="38"/>
-<contactref element="U$1" pad="19"/>
 <contactref element="IC1" pad="GND"/>
 <contactref element="SV4" pad="13"/>
@@
 <vertex x="124.46" y="90.17"/>
 </polygon>
-<wire x1="266.69" y1="180.14" x2="312.41" y2="157.49" width="0" layer="19" extent="1-1"/>
-<wire x1="86.36" y1="83.82" x2="266.69" y2="180.14" width="0" layer="19" extent="1-1"/>
 </signal>
 <signal name="N$4">
