File: circuit/schematics/cotroler.sch (EAGLE design)
At the start: 17 parts

Commit message: dekita
Parts:
- removed D1, D2: (no value), diode:DIODE-C1702-15
- removed R1, R3: 7kΩ, rcl:R-EU_0204/2V
- removed R2, R4: 5kΩ, rcl:R-EU_0204/2V
- added D3, D4: (no value), diode:DIODE-D-10
- added R6, R7, R8, R9: (no value), resistor:R-EU_0207/10
Connections:
- net GND: now also R7.2, R8.2; no longer R2.2, R4.2
- net N$1: now also R6.1; no longer R1.2
- net N$10: now also D3.C, D4.C; no longer D1.C, D2.C
- net N$4: now also R6.2, R7.1; no longer R1.1, R2.1
- net N$5: now also R9.1; no longer R3.1
- net N$6: now also R8.1, R9.2; no longer R3.2, R4.1
- net N$7: now also D4.A; no longer D2.A
- net N$8: now also D3.A; no longer D1.A
Other:
- moved on the sheet: U$1

Commit message: drc cleared
Parts:
- removed U$1: ESP32DEVKITC, ESP32-DEVKITC:ESP32DEVKITC
Connections:
- net GND: no longer U$1.5V, U$1.GND@38
Changed lines of the file:
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@@
 <part name="SV1" library="con-lsta" library_urn="urn:adsk.eagle:library:161" deviceset="FE08-1" device="" package3d_urn="urn:adsk.eagle:package:8194/1"/>
 <part name="SV2" library="con-lsta" library_urn="urn:adsk.eagle:library:161" deviceset="FE10-1" device="" package3d_urn="urn:adsk.eagle:package:8192/1"/>
-<part name="U$1" library="ESP32-DEVKITC" deviceset="ESP32DEVKITC" device=""/>
 <part name="SV3" library="con-lsta" library_urn="urn:adsk.eagle:library:161" deviceset="FE20-1" device="" package3d_urn="urn:adsk.eagle:package:8196/1"/>
 <part name="SV4" library="con-lsta" library_urn="urn:adsk.eagle:library:161" deviceset="FE20-1" device="" package3d_urn="urn:adsk.eagle:package:8196/1"/>
@@
 <attribute name="VALUE" x="133.35" y="17.78" size="1.778" layer="96"/>
 <attribute name="NAME" x="133.35" y="49.022" size="1.778" layer="95"/>
-</instance>
-<instance part="U$1" gate="G$1" x="-25.4" y="38.1" smashed="yes" rot="R270">
-<attribute name="NAME" x="-20.32" y="64.77" size="1.27" layer="95"/>
 </instance>
 <instance part="SV3" gate="G$1" x="86.36" y="22.86" smashed="yes">
@@
 <wire x1="111.76" y1="55.88" x2="111.76" y2="66.04" width="0.1524" layer="91"/>
 <pinref part="IC2" gate="1" pin="GND"/>
-<pinref part="U$1" gate="G$1" pin="GND@38"/>
-<pinref part="U$1" gate="G$1" pin="5V"/>
 <wire x1="99.06" y1="76.2" x2="99.06" y2="55.88" width="0.1524" layer="91"/>
 <pinref part="IC1" gate="1" pin="GND"/>
