File: circuit/schematics/test_brd_add_gnd.sch (EAGLE design)
At the start: 12 parts, among them Q1 2N5484, X1 JST-XH-02-PIN-LONG-PAD, X2 JST-XH-02-PIN-LONG-PAD, X3 JST-XH-05-PIN-LONG-PAD

Commit message: drc cleared
Parts:
- removed U$1: ESP32DEVKITC, ESP32-DEVKITC:ESP32DEVKITC
Changed lines of the file:
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@@
 </classes>
 <parts>
-<part name="U$1" library="ESP32-DEVKITC" deviceset="ESP32DEVKITC" device=""/>
 <part name="R1" library="resistor" library_urn="urn:adsk.eagle:library:348" deviceset="R-EU_" device="0207/10" package3d_urn="urn:adsk.eagle:package:25939/1" value="10kΩ"/>
 <part name="R2" library="resistor" library_urn="urn:adsk.eagle:library:348" deviceset="R-EU_" device="0207/10" package3d_urn="urn:adsk.eagle:package:25939/1" value="330Ω"/>
@@
 </plain>
 <instances>
-<instance part="U$1" gate="G$1" x="15.24" y="71.12" smashed="yes" rot="R90">
-<attribute name="NAME" x="10.16" y="44.45" size="1.27" layer="95" rot="R180"/>
-</instance>
 <instance part="R1" gate="G$1" x="73.66" y="66.04" smashed="yes">
 <attribute name="NAME" x="69.85" y="67.5386" size="1.778" layer="95"/>
